File: Strelka_Flight_Computer/ASM330LHHXTR.kicad_sch (KiCad schematic)
At the start: 4 parts, among them U1 ASM330LHHXTR

Commit message: Added LCSC mpn to all relevent parts
Parts:
- C30: LCSC (none) -> C1525
Changed lines of the file:
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@@
+      (effects (font (size 1.27 1.27)) hide)
+    )
+    (property "LCSC" " C1525" (at 179.324 115.062 0)
       (effects (font (size 1.27 1.27)) hide)
     )
@@
       (effects (font (size 1.27 1.27)) hide)
     )
+    (property "LCSC" " C1525" (at 116.078 106.426 0)
+      (effects (font (size 1.27 1.27)) hide)
+    )
