File: Strelka_Flight_Computer/Ematch.kicad_sch (KiCad schematic)
At the start: 12 parts, among them Q10 AP2300, Q11 MMBT2222, Q9 AO3401A

Commit message: Completely exported to JLC
Parts:
- C6: LCSC (none) -> C15195
Changed lines of the file:
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@@
+      (effects (font (size 1.27 1.27)) hide)
+    )
+    (property "LCSC" "C15195" (at 131.064 141.097 0)
       (effects (font (size 1.27 1.27)) hide)
     )
