File: Strelka_Flight_Computer/MAX-M10S-00B.kicad_sch (KiCad schematic)
At the start: 14 parts, among them IC2 MAX-M10S-00B

Commit message: Completely exported to JLC
Parts:
- C38: LCSC 2.2u -> C23733
Changed lines of the file:
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@@
       (effects (font (size 1.27 1.27)) hide)
     )
-    (property "LCSC" "2.2u" (at 57.785 157.48 0)
+    (property "LCSC" "C23733" (at 57.785 157.48 0)
       (effects (font (size 1.27 1.27)) hide)
     )
