File: Strelka_Flight_Computer/Power.kicad_sch (KiCad schematic)
At the start: 44 parts, among them J1 1S_LiPo_LARGE_HOLE_XT-30, Q1 CJK2333, Q2 CJK2333, SW3 SM02B-GHS-TB(LF)(SN), U16 TPS61085DGKR, U2 AP9101CK6, U3 AMS1117-3.3

Commit message: Started design for V2
Parts:
- removed C49, C50, C52, C53, C54: NC, Capacitor_SMD:C_0603_1608Metric, symbol Device:C_Small
- removed J1: 1S_LiPo_LARGE_HOLE_XT-30, Connector_AMASS:AMASS_XT30PW-M_1x02_P2.50mm_Horizontal, symbol Connector:Conn_01x02_Female
- removed SW3: SM02B-GHS-TB(LF)(SN), Footprints:SM02BGHSTBLFSN, symbol Switch:SW_DIP_x01
- added J1: Conn_01x02, Footprints:MOLEX_43045-0200, symbol Connector_Generic:Conn_01x02
- added SW1: SW_DIP_x01, Footprints:MOLEX_43045-0200, symbol Switch:SW_DIP_x01
Connections:
- net +BATT: now also J1.1 (Pin_1)
- net -BATT: now also J1.2 (Pin_2)
- net VDC: now also SW1.2
- net at D1.1 (K), Q1.2 (S): now also SW1.1
Other:
- note removed: "Bulk capacitance as back up"

Commit message: Routing starting
Parts:
- removed C57: NC, Capacitor_SMD:C_0805_2012Metric, symbol Device:C_Small
- removed C7: 100nF, Capacitor_SMD:C_0603_1608Metric_Pad1.08x0.95mm_HandSolder, symbol Device:C_Small
- removed C8, C9: 10uF, Capacitor_SMD:C_0603_1608Metric_Pad1.08x0.95mm_HandSolder, symbol Device:C_Small
- removed R20: 0, Resistor_SMD:R_0603_1608Metric, symbol Device:R_Small
- added C30 (x2): 10uF, Capacitor_SMD:C_0402_1005Metric, symbol Device:C_Small
- added C5: 100n, Capacitor_SMD:C_0402_1005Metric, symbol Device:C_Small
- added R1: NC, Resistor_SMD:R_0603_1608Metric, symbol Device:R_Small
- C47: footprint Capacitor_SMD:C_0603_1608Metric -> Capacitor_SMD:C_0402_1005Metric
- C48: value 0.1u -> 100n; footprint Capacitor_SMD:C_0603_1608Metric -> Capacitor_SMD:C_0402_1005Metric
- C51: value 820p -> 2.2n; footprint Capacitor_SMD:C_0603_1608Metric -> Capacitor_SMD:C_0402_1005Metric; LCSC (none) -> C1531
- C6: value 0.1uF -> 100n; footprint Capacitor_SMD:C_0603_1608Metric -> Capacitor_SMD:C_0402_1005Metric
- R3, R8: footprint Resistor_SMD:R_0603_1608Metric -> Resistor_SMD:R_0402_1005Metric; LCSC (none) -> C25741
- R61: value 56.2k -> 10k; footprint Resistor_SMD:R_0603_1608Metric -> Resistor_SMD:R_0402_1005Metric; LCSC# C105579 -> C25744
- R7: footprint Resistor_SMD:R_0603_1608Metric -> Resistor_SMD:R_0402_1005Metric; LCSC (none) -> C25104
Connections:
- net +3V3: now also C30.1, C30.1
- net +5V: now also C5.1
- net +5VA: now also Q2.3 (D)
- net GND: now also C30.2, C30.2, C5.2, R1.2

Commit message: Continued routing
Parts:
- R1: value NC -> 0R; now not fitted
Connections:
- net SW_IN: now reaches D1.1 (K), Q1.2 (S), SW1.1
Changed lines of the file:
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@@
+    (effects (font (size 1.27 1.27)) (justify left bottom))
+  )
+  (label "SW_IN" (at 77.724 48.26 0) (fields_autoplaced)
     (effects (font (size 1.27 1.27)) (justify left bottom))
   )
@@
   )
   (symbol (lib_id "Device:R_Small") (at 145.415 86.487 90) (unit 1)
-    (in_bom yes) (on_board yes) (dnp no) (fields_autoplaced)
+    (in_bom yes) (on_board yes) (dnp yes) (fields_autoplaced)
     (property "Reference" "R1" (at 145.415 82.296 90)
       (effects (font (size 1.27 1.27)))
     )
-    (property "Value" "NC" (at 145.415 84.836 90)
-      (effects (font (size 1.27 1.27)))
-    )
+    (property "Value" "0R" (at 145.415 84.836 90)
+      (effects (font (size 1.27 1.27)))
+    )

Commit message: Routing complete
Connections:
- net -BATT: now also R1.1
- net +3V3 renamed +3.3V
Changed lines of the file:
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@@
   (junction (at 231.14 132.08) (diameter 0) (color 0 0 0 0)
   )
+  (junction (at 213.106 35.56) (diameter 0) (color 0 0 0 0)
+  )
   (junction (at 68.58 57.15) (diameter 0) (color 0 0 0 0)
   )
@@
   (junction (at 129.54 151.13) (diameter 0) (color 0 0 0 0)
   )
+  (junction (at 121.92 74.93) (diameter 0) (color 0 0 0 0)
+  )
   (junction (at 125.73 55.88) (diameter 0) (color 0 0 0 0)
   )
@@
   )
   (junction (at 91.44 74.93) (diameter 0) (color 0 0 0 0)
-  )
-  (junction (at 213.36 35.56) (diameter 0) (color 0 0 0 0)
   )
   (junction (at 167.894 74.93) (diameter 0) (color 0 0 0 0)
@@
     (stroke (width 0) (type default))
   )
-  (wire (pts (xy 121.793 74.93) (xy 121.793 86.487))
+  (wire (pts (xy 121.92 74.93) (xy 121.92 86.487))
     (stroke (width 0) (type default))
   )
@@
     (stroke (width 0) (type default))
   )
-  (wire (pts (xy 121.793 86.487) (xy 142.875 86.487))
+  (wire (pts (xy 121.92 86.487) (xy 142.875 86.487))
     (stroke (width 0) (type default))
   )
@@
     (stroke (width 0) (type default))
   )
+  (wire (pts (xy 213.106 35.56) (xy 217.17 35.56))
+    (stroke (width 0) (type default))
+  )
   (wire (pts (xy 208.28 139.7) (xy 214.63 139.7))
-    (stroke (width 0) (type default))
-  )
-  (wire (pts (xy 209.55 35.56) (xy 213.36 35.56))
     (stroke (width 0) (type default))
   )
@@
     (stroke (width 0) (type solid))
   )
-  (wire (pts (xy 213.36 35.56) (xy 217.17 35.56))
+  (wire (pts (xy 209.55 35.56) (xy 213.106 35.56))
     (stroke (width 0) (type default))
   )
@@
     )
   )
+  (symbol (lib_name "+3.3V_1") (lib_id "power:+3.3V") (at 213.106 35.56 0) (unit 1)
+    (in_bom yes) (on_board yes) (dnp no) (fields_autoplaced)
+    (property "Reference" "#PWR015" (at 213.106 39.37 0)
+      (effects (font (size 1.27 1.27)) hide)
+    )
+    (property "Value" "+3.3V" (at 213.106 32.131 0)
+      (effects (font (size 1.27 1.27)))
+    )
+    (property "Footprint" "" (at 213.106 35.56 0)
+      (effects (font (size 1.27 1.27)) hide)
+    )
+    (property "Datasheet" "" (at 213.106 35.56 0)
+      (effects (font (size 1.27 1.27)) hide)
+    )
+    (pin "1")
+    (instances
+      (project "Strelka_Flight_Computer"
+        (path "/e63e39d7-6ac0-4ffd-8aa3-1841a4541b55/0daddb18-1491-4767-9ffd-66c8a8ce3cbd"
+          (reference "#PWR015") (unit 1)
+        )
+      )
+    )
+  )
   (symbol (lib_id "power:GND") (at 190.5 43.18 0) (unit 1)
     (in_bom yes) (on_board yes) (dnp no) (fields_autoplaced)
@@
         )
       )
-    )
-  )
-  (symbol (lib_id "power:+3.3V") (at 213.36 35.56 0) (unit 1)
-    (in_bom yes) (on_board yes) (dnp no) (fields_autoplaced)
-    (property "Reference" "#PWR0117" (at 213.36 39.37 0)
-      (effects (font (size 1.27 1.27)) hide)
-    )
-    (property "Value" "+3.3V" (at 213.36 31.9842 0)
-      (effects (font (size 1.27 1.27)))
-    )
-    (property "Footprint" "" (at 213.36 35.56 0)
-      (effects (font (size 1.27 1.27)) hide)
-    )
-    (property "Datasheet" "" (at 213.36 35.56 0)
-      (effects (font (size 1.27 1.27)) hide)
-    )
-    (pin "1")
-    (instances
-      (project "Strelka_Flight_Computer"
-        (path "/e63e39d7-6ac0-4ffd-8aa3-1841a4541b55/0daddb18-1491-4767-9ffd-66c8a8ce3cbd"
-          (reference "#PWR0117") (unit 1)
-        )
-      )

Commit message: Created BOM
Parts:
- C30: value 10uF -> 10u
- C41: LCSC (none) -> C248440; LCSC# C248440 -> (none)
- D1, D2, D4: LCSC (none) -> C8598; LCSC# C8598 -> (none)
- D13: LCSC (none) -> C2858499; LCSC# C2858499 -> (none)
- D14: LCSC (none) -> C908230; LCSC# C908230 -> (none)
- L2: LCSC (none) -> C1329837; LCSC# C1329837 -> (none)
- MOSFET1: LCSC (none) -> C151635; LCSC# C151635 -> (none)
- Q1: LCSC (none) -> C504109; LCSC# C504109 -> (none)
- Q2: footprint Package_TO_SOT_SMD:SOT-23 -> Q3; LCSC (none) -> C504109; LCSC# C504109 -> (none)
- R59: LCSC (none) -> C137796; LCSC# C137796 -> (none)
- R60, R62, R63: LCSC (none) -> C105579; LCSC# C105579 -> (none)
- R61: LCSC (none) -> C25744; LCSC# C25744 -> (none)
- U16: LCSC (none) -> C113659; LCSC# C113659 -> (none)
- U2: LCSC (none) -> C151339; LCSC# C151339 -> (none)
- U3: LCSC (none) -> C173386; LCSC# C173386 -> (none)
Changed lines of the file:
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@@
       (effects (font (size 1.27 1.27)) (justify left))
     )
-    (property "Value" "10uF" (at 212.09 39.37 0)
+    (property "Value" "10u" (at 212.09 39.37 0)
       (effects (font (size 1.27 1.27)) (justify left))
     )
@@
       (effects (font (size 1.27 1.27)) hide)
     )
-    (property "LCSC#" "C105579" (at 129.54 147.32 0)
+    (property "LCSC" "C105579" (at 129.54 147.32 0)
       (effects (font (size 1.27 1.27)) hide)
     )
@@
       (effects (font (size 1.27 1.27)) hide)
     )
-    (property "LCSC#" "C105579" (at 129.54 153.67 0)
+    (property "LCSC" "C105579" (at 129.54 153.67 0)
       (effects (font (size 1.27 1.27)) hide)
     )
@@
       (effects (font (size 1.524 1.524)) hide)
     )
-    (property "LCSC#" "C151635" (at 125.73 69.85 0)
+    (property "LCSC" "C151635" (at 125.73 69.85 0)
       (effects (font (size 1.27 1.27)) hide)
     )
@@
       (effects (font (size 1.27 1.27)) hide)
     )
-    (property "LCSC#" "C105579" (at 83.82 78.74 0)
+    (property "LCSC" "C105579" (at 83.82 78.74 0)
       (effects (font (size 1.27 1.27)) hide)
     )
@@
       (effects (font (size 1.27 1.27)) hide)
     )
-    (property "LCSC#" "C8598" (at 201.93 139.7 0)
+    (property "LCSC" "C8598" (at 201.93 139.7 0)
       (effects (font (size 1.27 1.27)) hide)
     )
@@
       (effects (font (size 1.27 1.27)) (justify left))
     )
-    (property "Footprint" "Package_TO_SOT_SMD:SOT-23" (at 216.535 129.54 0)
+    (property "Footprint" "Q3" (at 216.535 129.54 0)
       (effects (font (size 1.27 1.27) italic) (justify left) hide)
     )
@@
       (effects (font (size 1.27 1.27)) (justify left) hide)
     )
-    (property "LCSC#" "C504109" (at 214.63 134.62 0)
+    (property "LCSC" "C504109" (at 214.63 134.62 0)
       (effects (font (size 1.27 1.27)) hide)
     )
@@
       (effects (font (size 1.27 1.27)) hide)
     )
-    (property "LCSC#" "C25744" (at 113.03 154.94 0)
+    (property "LCSC" "C25744" (at 113.03 154.94 0)
       (effects (font (size 1.27 1.27)) hide)
     )
@@
       (effects (font (size 1.27 1.27)) (justify left bottom) hide)
     )
-    (property "LCSC#" "C113659" (at 97.79 140.335 0)
+    (property "LCSC" "C113659" (at 97.79 140.335 0)
       (effects (font (size 1.27 1.27)) (justify left bottom) hide)
     )
@@
       (effects (font (size 1.27 1.27)) hide)
     )
-    (property "LCSC#" "C1329837" (at 91.44 133.35 90)
+    (property "LCSC" "C1329837" (at 91.44 133.35 90)
       (effects (font (size 1.27 1.27)) hide)
     )
@@
       (effects (font (size 1.27 1.27)) hide)
     )
-    (property "LCSC#" "C8598" (at 85.09 53.34 90)
+    (property "LCSC" "C8598" (at 85.09 53.34 90)
       (effects (font (size 1.27 1.27)) hide)
     )
@@
       (effects (font (size 1.27 1.27)) (justify left))
     )
-    (property "Value" "10uF" (at 219.71 39.37 0)
+    (property "Value" "10u" (at 219.71 39.37 0)
       (effects (font (size 1.27 1.27)) (justify left))
     )
@@
       (effects (font (size 1.27 1.27)) (justify left) hide)
     )
-    (property "LCSC#" "C504109" (at 68.58 50.8 0)
+    (property "LCSC" "C504109" (at 68.58 50.8 0)
       (effects (font (size 1.27 1.27)) hide)
     )
@@
       (effects (font (size 1.27 1.27)) hide)
     )
-    (property "LCSC#" "C173386" (at 201.93 35.56 0)
+    (property "LCSC" "C173386" (at 201.93 35.56 0)
       (effects (font (size 1.27 1.27)) hide)
     )
@@
       (effects (font (size 1.27 1.27)) hide)
     )
-    (property "LCSC#" "C151339" (at 146.05 48.26 0)
+    (property "LCSC" "C151339" (at 146.05 48.26 0)
       (effects (font (size 1.27 1.27)) hide)
     )
@@
       (effects (font (size 1.27 1.27)) hide)
     )
-    (property "LCSC#" "C8598" (at 231.14 137.16 90)
+    (property "LCSC" "C8598" (at 231.14 137.16 90)
       (effects (font (size 1.27 1.27)) hide)
     )
@@
       (effects (font (size 1.27 1.27)) hide)
     )
-    (property "LCSC#" "C908230" (at 119.38 143.51 0)
+    (property "LCSC" "C908230" (at 119.38 143.51 0)
       (effects (font (size 1.27 1.27)) hide)
     )
@@
       (effects (font (size 1.27 1.27)) hide)
     )
-    (property "LCSC#" "C137796" (at 83.82 71.12 0)
+    (property "LCSC" "C137796" (at 83.82 71.12 0)
       (effects (font (size 1.27 1.27)) hide)
     )
@@
       (effects (font (size 1.27 1.27)) hide)
     )
-    (property "LCSC#" "C248440" (at 101.6 54.61 0)
+    (property "LCSC" "C248440" (at 101.6 54.61 0)
       (effects (font (size 1.27 1.27)) hide)
     )
@@
       (effects (font (size 1.27 1.27)) hide)
     )
-    (property "LCSC#" "C2858499" (at 91.44 78.74 90)
-      (effects (font (size 1.27 1.27)) hide)
-    )
+    (property "LCSC" "C2858499" (at 91.44 78.74 90)
+      (effects (font (size 1.27 1.27)) hide)
+    )

Commit message: Added lp filter caps to adc signals
Parts:
- added C9: 10n, Capacitor_SMD:C_0402_1005Metric, symbol Device:C_Small
Connections:
- net BATT_VOLT: now also C9.1
- net GND: now also C9.2
Other:
- note added: "LP filter BW 1.22kHz"
- moved on the sheet: D13
Changed lines of the file:
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@@
   (junction (at 213.106 35.56) (diameter 0) (color 0 0 0 0)
   )
+  (junction (at 94.869 74.93) (diameter 0) (color 0 0 0 0)
+  )
   (junction (at 68.58 57.15) (diameter 0) (color 0 0 0 0)
   )
+  (junction (at 87.757 82.55) (diameter 0) (color 0 0 0 0)
+  )
   (junction (at 190.5 35.56) (diameter 0) (color 0 0 0 0)
   )
@@
   (junction (at 85.09 48.26) (diameter 0) (color 0 0 0 0)
   )
+  (junction (at 87.757 74.93) (diameter 0) (color 0 0 0 0)
+  )
   (junction (at 101.6 48.26) (diameter 0) (color 0 0 0 0)
   )
@@
   )
   (junction (at 153.67 40.64) (diameter 1.016) (color 0 0 0 0)
-  )
-  (junction (at 91.44 74.93) (diameter 0) (color 0 0 0 0)
   )
   (junction (at 167.894 74.93) (diameter 0) (color 0 0 0 0)
@@
     (stroke (width 0) (type solid))
   )
+  (wire (pts (xy 87.757 74.93) (xy 94.869 74.93))
+    (stroke (width 0) (type default))
+  )
   (wire (pts (xy 209.55 43.18) (xy 213.36 43.18))
     (stroke (width 0) (type default))
@@
     (stroke (width 0) (type default))
   )
+  (wire (pts (xy 87.757 81.026) (xy 87.757 82.55))
+    (stroke (width 0) (type default))
+  )
   (wire (pts (xy 121.92 74.93) (xy 121.92 86.487))
     (stroke (width 0) (type default))
@@
   )
   (polyline (pts (xy 179.07 109.22) (xy 238.76 109.22))
+    (stroke (width 0) (type default))
+  )
+  (wire (pts (xy 87.757 82.55) (xy 94.869 82.55))
     (stroke (width 0) (type default))
   )
@@
     (stroke (width 0) (type solid))
   )
+  (wire (pts (xy 94.869 74.93) (xy 96.012 74.93))
+    (stroke (width 0) (type default))
+  )
   (wire (pts (xy 132.08 29.21) (xy 171.45 29.21))
     (stroke (width 0) (type solid))
@@
     (stroke (width 0) (type default))
   )
-  (wire (pts (xy 83.82 74.93) (xy 91.44 74.93))
+  (wire (pts (xy 83.82 74.93) (xy 87.757 74.93))
     (stroke (width 0) (type default))
   )
@@
     (stroke (width 0) (type default))
   )
-  (wire (pts (xy 91.44 74.93) (xy 95.25 74.93))
-    (stroke (width 0) (type default))
-  )
   (wire (pts (xy 80.01 165.1) (xy 105.41 165.1))
     (stroke (width 0) (type default))
@@
     (stroke (width 0) (type solid))
   )
-  (wire (pts (xy 91.44 82.55) (xy 91.44 81.28))
+  (wire (pts (xy 94.869 82.55) (xy 94.869 81.28))
     (stroke (width 0) (type default))
   )
@@
     (stroke (width 0) (type default))
   )
-  (wire (pts (xy 83.82 82.55) (xy 91.44 82.55))
+  (wire (pts (xy 83.82 82.55) (xy 87.757 82.55))
     (stroke (width 0) (type default))
   )
@@
   )
   (wire (pts (xy 208.28 139.7) (xy 214.63 139.7))
+    (stroke (width 0) (type default))
+  )
+  (wire (pts (xy 87.757 74.93) (xy 87.757 75.946))
     (stroke (width 0) (type default))
   )
@@
     (stroke (width 0) (type default))
   )
-  (wire (pts (xy 91.44 76.2) (xy 91.44 74.93))
+  (wire (pts (xy 94.869 76.2) (xy 94.869 74.93))
     (stroke (width 0) (type default))
   )
@@
     (effects (font (size 1.27 1.27)) (justify left bottom))
   )
+  (text "LP filter BW\n1.22kHz" (at 87.503 87.249 0)
+    (effects (font (size 1.27 1.27)) (justify left bottom))
+  )
   (text "BATTERY PROTECTION" (at 137.1854 25.1206 0)
     (effects (font (size 1.27 1.27)) (justify left bottom))
@@
     (effects (font (size 1.27 1.27)) (justify left bottom))
   )
-  (hierarchical_label "BATT_VOLT" (shape input) (at 95.25 74.93 0) (fields_autoplaced)
+  (hierarchical_label "BATT_VOLT" (shape input) (at 96.012 74.93 0) (fields_autoplaced)
     (effects (font (size 1.27 1.27)) (justify left))
   )
@@
     )
   )
+  (symbol (lib_id "Device:C_Small") (at 87.757 78.486 0) (unit 1)
+    (in_bom yes) (on_board yes) (dnp no)
+    (property "Reference" "C9" (at 89.662 77.6001 0)
+      (effects (font (size 1.27 1.27)) (justify left))
+    )
+    (property "Value" "10n" (at 89.662 80.137 0)
+      (effects (font (size 1.27 1.27)) (justify left))
+    )
+    (property "Footprint" "Capacitor_SMD:C_0402_1005Metric" (at 87.757 78.486 0)
+      (effects (font (size 1.27 1.27)) hide)
+    )
+    (property "Datasheet" "~" (at 87.757 78.486 0)
+      (effects (font (size 1.27 1.27)) hide)
+    )
+    (pin "1")
+    (pin "2")
+    (instances
+      (project "Strelka_Flight_Computer"
+        (path "/e63e39d7-6ac0-4ffd-8aa3-1841a4541b55/0daddb18-1491-4767-9ffd-66c8a8ce3cbd"
+          (reference "C9") (unit 1)
+        )
+      )
+    )
+  )
   (symbol (lib_id "Transistor_FET:Si2319CDS") (at 68.58 50.8 90) (unit 1)
     (in_bom yes) (on_board yes) (dnp no)
@@
     )
   )
-  (symbol (lib_id "Device:D_Zener_Small_Filled") (at 91.44 78.74 270) (unit 1)
-    (in_bom yes) (on_board yes) (dnp no) (fields_autoplaced)
-    (property "Reference" "D13" (at 93.98 77.4699 90)
-      (effects (font (size 1.27 1.27)) (justify left))
-    )
-    (property "Value" "BZT52C3V6T" (at 93.98 80.0099 90)
-      (effects (font (size 1.27 1.27)) (justify left))
-    )
-    (property "Footprint" "Diode_SMD:D_SOD-523" (at 91.44 78.74 90)
-      (effects (font (size 1.27 1.27)) hide)
-    )
-    (property "Datasheet" "https://datasheet.lcsc.com/lcsc/2108150230_MDD-Microdiode-Electronics--BZT52C3V6T_C2858499.pdf" (at 91.44 78.74 90)
-      (effects (font (size 1.27 1.27)) hide)
-    )
-    (property "LCSC" "C2858499" (at 91.44 78.74 90)
-      (effects (font (size 1.27 1.27)) hide)
-    )
+  (symbol (lib_id "Device:D_Zener_Small_Filled") (at 94.869 78.74 270) (unit 1)
+    (in_bom yes) (on_board yes) (dnp no) (fields_autoplaced)
+    (property "Reference" "D13" (at 97.409 77.4699 90)
+      (effects (font (size 1.27 1.27)) (justify left))
+    )
+    (property "Value" "BZT52C3V6T" (at 97.409 80.0099 90)
+      (effects (font (size 1.27 1.27)) (justify left))
+    )
+    (property "Footprint" "Diode_SMD:D_SOD-523" (at 94.869 78.74 90)
+      (effects (font (size 1.27 1.27)) hide)
+    )
+    (property "Datasheet" "https://datasheet.lcsc.com/lcsc/2108150230_MDD-Microdiode-Electronics--BZT52C3V6T_C2858499.pdf" (at 94.869 78.74 90)
+      (effects (font (size 1.27 1.27)) hide)
+    )
+    (property "LCSC" "C2858499" (at 94.869 78.74 90)
+      (effects (font (size 1.27 1.27)) hide)
+    )
