File: Strelka_Flight_Computer/Power.kicad_sch (KiCad schematic)
At the start: 39 parts, among them J1 Conn_01x02, Q1 CJK2333, Q2 CJK2333, SW1 SW_DIP_x01, U16 TPS61085DGKR, U2 AP9101CK6, U3 AMS1117-3.3

Commit message: Added LCSC mpn to all relevent parts
Parts:
- removed C56: 47u, Capacitor_SMD:C_0805_2012Metric, symbol Device:C_Small
- added C14: 22u, Capacitor_SMD:C_0805_2012Metric, symbol Device:C_Small
- C46: LCSC (none) -> C59461
- C47: LCSC (none) -> C52923
- C48, C5, C6: LCSC (none) -> C1525
- C55: value 47u -> 22u; LCSC (none) -> C45783
- Q2: footprint Q3 -> Package_TO_SOT_SMD:SOT-23
- R59: LCSC C137796 -> C22797
- R62: LCSC C105579 -> C23254
- R63: LCSC C105579 -> C22967
- R9: LCSC (none) -> C13167
Connections:
- net +5VA: now also C14.1
- net GND: now also C14.2
Changed lines of the file:
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@@
+      (effects (font (size 1.27 1.27)) hide)
+    )
+    (property "LCSC" " C1525" (at 80.01 161.29 0)
       (effects (font (size 1.27 1.27)) hide)
     )
@@
     )
     (property "Datasheet" "~" (at 66.04 149.86 0)
+      (effects (font (size 1.27 1.27)) hide)
+    )
+    (property "LCSC" " C52923" (at 66.04 149.86 0)
       (effects (font (size 1.27 1.27)) hide)
     )
@@
       (effects (font (size 1.27 1.27)) hide)
     )
-    (property "LCSC" "C105579" (at 129.54 147.32 0)
+    (property "LCSC" "C23254" (at 129.54 147.32 0)
       (effects (font (size 1.27 1.27)) hide)
     )
@@
       (effects (font (size 1.27 1.27)) hide)
     )
-    (property "LCSC" "C105579" (at 129.54 153.67 0)
+    (property "LCSC" "C22967" (at 129.54 153.67 0)
       (effects (font (size 1.27 1.27)) hide)
     )
@@
       (effects (font (size 1.27 1.27)) hide)
     )
+    (property "LCSC" "C13167" (at 171.45 71.12 0)
+      (effects (font (size 1.27 1.27)) hide)
+    )
     (pin "1")
     (pin "2")
@@
       (effects (font (size 1.27 1.27)) (justify left))
     )
-    (property "Footprint" "Q3" (at 216.535 129.54 0)
+    (property "Footprint" "Package_TO_SOT_SMD:SOT-23" (at 216.535 129.54 0)
       (effects (font (size 1.27 1.27) italic) (justify left) hide)
     )
@@
     )
   )
+  (symbol (lib_id "Device:C_Small") (at 148.59 149.86 0) (unit 1)
+    (in_bom yes) (on_board yes) (dnp no) (fields_autoplaced)
+    (property "Reference" "C14" (at 150.9141 149.0316 0)
+      (effects (font (size 1.27 1.27)) (justify left))
+    )
+    (property "Value" "22u" (at 150.9141 151.5685 0)
+      (effects (font (size 1.27 1.27)) (justify left))
+    )
+    (property "Footprint" "Capacitor_SMD:C_0805_2012Metric" (at 148.59 149.86 0)
+      (effects (font (size 1.27 1.27)) hide)
+    )
+    (property "Datasheet" "~" (at 148.59 149.86 0)
+      (effects (font (size 1.27 1.27)) hide)
+    )
+    (property "LCSC" "C45783" (at 148.59 149.86 0)
+      (effects (font (size 1.27 1.27)) hide)
+    )
+    (pin "1")
+    (pin "2")
+    (instances
+      (project "Strelka_Flight_Computer"
+        (path "/e63e39d7-6ac0-4ffd-8aa3-1841a4541b55/0daddb18-1491-4767-9ffd-66c8a8ce3cbd"
+          (reference "C14") (unit 1)
+        )
+      )
+    )
+  )
   (symbol (lib_name "+3.3V_1") (lib_id "power:+3.3V") (at 213.106 35.56 0) (unit 1)
     (in_bom yes) (on_board yes) (dnp no) (fields_autoplaced)
@@
     )
     (property "Datasheet" "~" (at 163.83 44.45 0)
+      (effects (font (size 1.27 1.27)) hide)
+    )
+    (property "LCSC" " C1525" (at 163.83 44.45 0)
       (effects (font (size 1.27 1.27)) hide)
     )
@@
         (path "/e63e39d7-6ac0-4ffd-8aa3-1841a4541b55/0daddb18-1491-4767-9ffd-66c8a8ce3cbd"
           (reference "C8") (unit 1)
-        )
-      )
-    )
-  )
-  (symbol (lib_id "Device:C_Small") (at 148.59 149.86 0) (unit 1)
-    (in_bom yes) (on_board yes) (dnp no) (fields_autoplaced)
-    (property "Reference" "C56" (at 150.9141 149.0316 0)
-      (effects (font (size 1.27 1.27)) (justify left))
-    )
-    (property "Value" "47u" (at 150.9141 151.5685 0)
-      (effects (font (size 1.27 1.27)) (justify left))
-    )
-    (property "Footprint" "Capacitor_SMD:C_0805_2012Metric" (at 148.59 149.86 0)
-      (effects (font (size 1.27 1.27)) hide)
-    )
-    (property "Datasheet" "~" (at 148.59 149.86 0)
-      (effects (font (size 1.27 1.27)) hide)
-    )
-    (pin "1")
-    (pin "2")
-    (instances
-      (project "Strelka_Flight_Computer"
-        (path "/e63e39d7-6ac0-4ffd-8aa3-1841a4541b55/0daddb18-1491-4767-9ffd-66c8a8ce3cbd"
-          (reference "C56") (unit 1)
         )
       )
@@
       (effects (font (size 1.27 1.27)) hide)
     )
+    (property "LCSC" "C59461" (at 55.88 149.86 0)
+      (effects (font (size 1.27 1.27)) hide)
+    )
     (pin "1")
     (pin "2")
@@
       (effects (font (size 1.27 1.27)) (justify left))
     )
-    (property "Value" "47u" (at 142.0241 151.5685 0)
+    (property "Value" "22u" (at 142.0241 151.5685 0)
       (effects (font (size 1.27 1.27)) (justify left))
     )
@@
       (effects (font (size 1.27 1.27)) hide)
     )
+    (property "LCSC" "C45783" (at 139.7 149.86 0)
+      (effects (font (size 1.27 1.27)) hide)
+    )
     (pin "1")
     (pin "2")
@@
       (effects (font (size 1.27 1.27)) hide)
     )
+    (property "LCSC" " C1525" (at 190.5 38.1 0)
+      (effects (font (size 1.27 1.27)) hide)
+    )
     (pin "1")
     (pin "2")
@@
       (effects (font (size 1.27 1.27)) hide)
     )
-    (property "LCSC" "C137796" (at 83.82 71.12 0)
-      (effects (font (size 1.27 1.27)) hide)
-    )
+    (property "LCSC" "C22797" (at 83.82 71.12 0)
+      (effects (font (size 1.27 1.27)) hide)
+    )

Commit message: Completely exported to JLC
Parts:
- C9: LCSC (none) -> C15195
- R60: LCSC C105579 -> C25819
- R63: LCSC C22967 -> C22967
Changed lines of the file:
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@@
       (effects (font (size 1.27 1.27)) hide)
     )
-    (property "LCSC" "C22967" (at 129.54 153.67 0)
+    (property "LCSC" " C22967" (at 129.54 153.67 0)
       (effects (font (size 1.27 1.27)) hide)
     )
@@
       (effects (font (size 1.27 1.27)) hide)
     )
-    (property "LCSC" "C105579" (at 83.82 78.74 0)
+    (property "LCSC" "C25819" (at 83.82 78.74 0)
       (effects (font (size 1.27 1.27)) hide)
     )
@@
       (effects (font (size 1.27 1.27)) hide)
     )
+    (property "LCSC" "C15195" (at 87.757 78.486 0)
+      (effects (font (size 1.27 1.27)) hide)
+    )
