File: Strelka_Flight_Computer/Data_Interfaces.kicad_sch (KiCad schematic)
At the start: 3 parts, among them J2 SM04B-GHS-TB(LF)(SN)-, J6 USB_B_Micro, U8 USBLC6-2SC6

Commit message: Started design for V2
Parts:
- removed J2: SM04B-GHS-TB(LF)(SN)-, Footprints:JST_SM04B-GHS-TB(LF)(SN)-, symbol SM04B-GHS-TB_LF__SN_-:SM04B-GHS-TB(LF)(SN)-
- added C35: 100n, Capacitor_SMD:C_0402_1005Metric, symbol Device:C_Small
- added J16: Conn_01x04, Footprints:JST_SM04B-GHS-TB(LF)(SN)-, symbol Connector_Generic:Conn_01x06
- added JP7: UART_Switch, Footprints:UART_Switch, symbol UART_Switch:UART_Switch
- added R51: 1k, Resistor_SMD:R_0402_1005Metric, symbol Device:R_Small
- added R52: 120R, Resistor_SMD:R_0402_1005Metric, symbol Device:R_Small
- added U8: MCP2551-I-SN, Package_SO:SOIC-8_3.9x4.9mm_P1.27mm, symbol Interface_CAN_LIN:MCP2551-I-SN
Connections:
- net GND: now also C35.2, J16.1 (Pin_1), J16.4 (Pin_4), J16.5 (Pin_5), J16.6 (Pin_6), R51.2, U8.2 (VSS)
- new net: JP7.1 (RX1), U8.1 (TXD)
- new net: JP7.2 (TX1), U8.4 (RXD)
- new net: R51.1, U8.8 (Rs)
- new net +5V: C35.1, U8.3 (VDD)
- new net CAN_+: J16.2 (Pin_2), R52.1, U8.7 (CANH)
- new net CAN_-: J16.3 (Pin_3), R52.2, U8.6 (CANL)
- new net CAN_RXD: JP7.3 (TX2)
- new net CAN_TXD: JP7.4 (RX2)
- no-connect marks 1 -> 2
Other:
- note added: "Vref????"
- note removed: "SWD Programming Interface"
- moved on the sheet: J6, U8

Commit message: Routing starting
Changed lines of the file:
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@@
     (effects (font (size 1.27 1.27)) (justify right bottom))
   )
-  (hierarchical_label "CAN_RXD" (shape input) (at 81.4569 121.285 180) (fields_autoplaced)
+  (hierarchical_label "CAN_RXD" (shape input) (at 81.28 121.285 180) (fields_autoplaced)
     (effects (font (size 1.27 1.27)) (justify right))
   )

Commit message: Continued routing
Parts:
- added F1: MF-PSHT035KX-2, Resistor_SMD:R_0805_2012Metric, symbol Device:Polyfuse_Small
Connections:
- net +5V: now also F1.1
- net GND: no longer J16.1 (Pin_1)
- new net V_CAN: F1.2, J16.1 (Pin_1)
Changed lines of the file:
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@@
 (kicad_sch (version 20230121) (generator eeschema)
   (paper "A4")
-  (junction (at 180.34 127.635) (diameter 0) (color 0 0 0 0)
-  )
   (junction (at 182.88 130.175) (diameter 0) (color 0 0 0 0)
   )
@@
     (stroke (width 0) (type default))
   )
+  (wire (pts (xy 180.34 120.015) (xy 180.34 114.427))
+    (stroke (width 0) (type default))
+  )
   (wire (pts (xy 133.35 79.375) (xy 143.51 79.375))
     (stroke (width 0) (type default))
@@
     (stroke (width 0) (type default))
   )
-  (wire (pts (xy 180.34 127.635) (xy 180.34 120.015))
-    (stroke (width 0) (type default))
-  )
   (wire (pts (xy 173.99 121.285) (xy 173.99 122.555))
     (stroke (width 0) (type default))
@@
     (stroke (width 0) (type default))
   )
+  (wire (pts (xy 165.227 114.427) (xy 173.863 114.427))
+    (stroke (width 0) (type default))
+  )
   (wire (pts (xy 173.99 122.555) (xy 182.88 122.555))
     (stroke (width 0) (type default))
@@
     (stroke (width 0) (type default))
   )
+  (wire (pts (xy 165.227 113.538) (xy 165.227 114.427))
+    (stroke (width 0) (type default))
+  )
   (wire (pts (xy 128.27 69.215) (xy 133.35 69.215))
     (stroke (width 0) (type default))
@@
   )
   (wire (pts (xy 106.68 121.285) (xy 114.3 121.285))
+    (stroke (width 0) (type default))
+  )
+  (wire (pts (xy 178.943 114.427) (xy 180.34 114.427))
     (stroke (width 0) (type default))
   )
@@
     (effects (font (size 1.27 1.27)) (justify left bottom))
   )
+  (label "CAN_P" (at 84.328 118.745 0) (fields_autoplaced)
+    (effects (font (size 1.27 1.27)) (justify left bottom))
+  )
   (label "USB2_D+" (at 133.35 59.055 0) (fields_autoplaced)
     (effects (font (size 1.27 1.27)) (justify left bottom))
   )
+  (label "CAN_N" (at 84.455 121.285 0) (fields_autoplaced)
+    (effects (font (size 1.27 1.27)) (justify left bottom))
+  )
   (label "CAN_-" (at 168.91 126.365 180) (fields_autoplaced)
     (effects (font (size 1.27 1.27)) (justify right bottom))
   )
+  (label "V_CAN" (at 180.34 115.951 0) (fields_autoplaced)
+    (effects (font (size 1.27 1.27)) (justify left bottom))
+  )
   (label "CAN_+" (at 168.91 121.285 180) (fields_autoplaced)
     (effects (font (size 1.27 1.27)) (justify right bottom))
@@
   (hierarchical_label "USB_D+" (shape input) (at 160.02 59.055 0) (fields_autoplaced)
     (effects (font (size 1.27 1.27)) (justify left))
+  )
+  (symbol (lib_id "power:+5V") (at 165.227 113.538 0) (unit 1)
+    (in_bom yes) (on_board yes) (dnp no) (fields_autoplaced)
+    (property "Reference" "#PWR0202" (at 165.227 117.348 0)
+      (effects (font (size 1.27 1.27)) hide)
+    )
+    (property "Value" "+5V" (at 165.227 108.458 0)
+      (effects (font (size 1.27 1.27)))
+    )
+    (property "Footprint" "" (at 165.227 113.538 0)
+      (effects (font (size 1.27 1.27)) hide)
+    )
+    (property "Datasheet" "" (at 165.227 113.538 0)
+      (effects (font (size 1.27 1.27)) hide)
+    )
+    (pin "1")
+    (instances
+      (project "Strelka_Power_Board"
+        (path "/83158c8b-22ee-48c3-a78a-e95d14e6b912/3958b393-7ce3-4f40-b277-b0fcd5b28e2a"
+          (reference "#PWR0202") (unit 1)
+        )
+      )
+      (project "Strelka_Flight_Computer"
+        (path "/e63e39d7-6ac0-4ffd-8aa3-1841a4541b55/f1926e02-3170-4727-853e-1c4f3bbf137d"
+          (reference "#PWR014") (unit 1)
+        )
+      )
+    )
   )
   (symbol (lib_id "Interface_CAN_LIN:MCP2551-I-SN") (at 127 123.825 0) (unit 1)
@@
         )
       )
+    )
+  )
+  (symbol (lib_id "Device:Polyfuse_Small") (at 176.403 114.427 90) (unit 1)
+    (in_bom yes) (on_board yes) (dnp no) (fields_autoplaced)
+    (property "Reference" "F1" (at 176.403 109.22 90)
+      (effects (font (size 1.27 1.27)))
+    )
+    (property "Value" "MF-PSHT035KX-2" (at 176.403 111.76 90)
+      (effects (font (size 1.27 1.27)))
+    )
+    (property "Footprint" "Resistor_SMD:R_0805_2012Metric" (at 181.483 113.157 0)
+      (effects (font (size 1.27 1.27)) (justify left) hide)
+    )
+    (property "Datasheet" "https://datasheet.lcsc.com/lcsc/2202032000_BOURNS-MF-PSHT035KX-2_C2153979.pdf" (at 176.403 114.427 0)
+      (effects (font (size 1.27 1.27)) hide)
+    )
+    (property "LCSC" "C2153979" (at 176.403 114.427 90)
+      (effects (font (size 1.27 1.27)) hide)
+    )
+    (pin "1")
+    (pin "2")
+    (instances
+      (project "Strelka_Flight_Computer"
+        (path "/e63e39d7-6ac0-4ffd-8aa3-1841a4541b55/f1926e02-3170-4727-853e-1c4f3bbf137d"
+          (reference "F1") (unit 1)
+        )
+      )

Commit message: Created BOM
Parts:
- U8: LCSC (none) -> C2687116; LCSC# C2687116 -> (none)
Changed lines of the file:
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@@
       (effects (font (size 1.27 1.27)) hide)
     )
-    (property "LCSC#" "C2687116" (at 146.05 69.215 90)
+    (property "LCSC" "C2687116" (at 146.05 69.215 90)
       (effects (font (size 1.27 1.27)) hide)
     )

Commit message: Added LCSC mpn to all relevent parts
Parts:
- C35: LCSC (none) -> C1525
- R51: LCSC (none) -> C11702
- R52: LCSC (none) -> C25079
Changed lines of the file:
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@@
+      (effects (font (size 1.27 1.27)) hide)
+    )
+    (property "LCSC" " C1525" (at 157.48 103.505 0)
       (effects (font (size 1.27 1.27)) hide)
     )
@@
     )
     (property "Datasheet" "~" (at 149.86 123.825 0)
+      (effects (font (size 1.27 1.27)) hide)
+    )
+    (property "LCSC" "C25079" (at 149.86 123.825 0)
       (effects (font (size 1.27 1.27)) hide)
     )
@@
       (effects (font (size 1.27 1.27)) hide)
     )
+    (property "LCSC" " C11702" (at 107.95 132.715 0)
+      (effects (font (size 1.27 1.27)) hide)
+    )

Commit message: Finalised BOM and sent order:
Parts:
- removed JP7: UART_Switch, Footprints:UART_Switch, symbol UART_Switch:UART_Switch
- added C35: 4.7n, Capacitor_SMD:C_0603_1608Metric, symbol Device:C_Small
- added D6: SP0504BAJT, Package_TO_SOT_SMD:SOT-353_SC-70-5, symbol Power_Protection:SP0504BAJT
- added FL1: 744231121, Footprints:CHIP_31121_WRE, symbol Filter:Choke_Schaffner_RN102-0.3-02-12M
- added R52: 60R4, Resistor_SMD:R_0402_1005Metric, symbol Device:R_Small
- R52: value 120R -> 60R4; LCSC C25079 -> C241122
Connections:
- net CAN_+: now also D6.4 (K), FL1.3; no longer U8.7 (CANH)
- net CAN_-: now also D6.5 (K), FL1.1, R52.2; no longer R52.2, U8.6 (CANL)
- net CAN_RXD: now also U8.4 (RXD)
- net CAN_TXD: now also U8.1 (TXD)
- net GND: now also C35.2, D6.2 (A)
- new net CANH: FL1.4, U8.7 (CANH)
- new net CANL: FL1.2, U8.6 (CANL)
- new net tap: C35.1, R52.1, R52.2
- no-connect marks 2 -> 4
Other:
- moved on the sheet: C35, R51, R52, U8
