File: Strelka_Flight_Computer/STM32H743.kicad_sch (KiCad schematic)
At the start: 40 parts, among them J3 Conn_01x07, Q3 AO3400A, Q4 AO3400A, Q5 AO3401A, SW2 TS-1185-C-A-A-A, SW3 TS-1185-C-A-A-A, U6 STM32H743VITx, Y1 Q13FC1350000400, Y2 X1E0000210834

Commit message: Adj to BOM
Parts:
- C30: LCSC C1644 -> C1548
Changed lines of the file:
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@@
       (effects (font (size 1.27 1.27)) hide)
     )
-    (property "LCSC" "C1644" (at 257.302 33.782 0)
+    (property "LCSC" "C1548" (at 257.302 33.782 0)
+      (effects (font (size 1.27 1.27)) hide)
+    )
+    (property "Field5" "" (at 257.302 33.782 0)
       (effects (font (size 1.27 1.27)) hide)
     )
@@
       (effects (font (size 1.27 1.27)) hide)
     )
-    (property "LCSC" "C1644" (at 244.602 33.782 0)
-      (effects (font (size 1.27 1.27)) hide)
-    )
+    (property "LCSC" "C1548" (at 244.602 33.782 0)
+      (effects (font (size 1.27 1.27)) hide)
+    )
